Commit message: small directory changes
Got rid of the colab_test since I got it figured out, also made the paths in the URDF file relative so it would work with Colab

File: sebastian_v2.urdf (robot description, URDF)
Before this commit: robot sebastian, 27 links, 26 joints
Links:
- link back_left_p1: geometry collision mesh filename=cad_files//simulation//stls//back_left_p1_coarse.stl scale=0.001 0.001 0.001; visual mesh filename=cad_files//simulation//stls//back_left_p1_fine.stl scale=0.001 0.001 0.001
- link back_left_p2: geometry collision mesh filename=cad_files//simulation//stls//back_left_p2_coarse.stl scale=.001 .001 .001; visual mesh filename=cad_files//simulation//stls//back_left_p2_fine.stl scale=.001 .001 .001
- link back_left_p3: geometry collision mesh filename=cad_files//simulation//stls//back_left_p3_coarse.stl scale=.001 .001 .001; visual mesh filename=cad_files//simulation//stls//back_left_p3_fine.stl scale=.001 .001 .001
- link back_left_p4: geometry collision mesh filename=cad_files//simulation//stls//back_left_p4_coarse.stl scale=.001 .001 .001; visual mesh filename=cad_files//simulation//stls//back_left_p4_fine.stl scale=.001 .001 .001
- link back_right_p1: geometry collision mesh filename=cad_files//simulation//stls//back_right_p1_coarse.stl scale=0.001 0.001 0.001; visual mesh filename=cad_files//simulation//stls//back_right_p1_fine.stl scale=0.001 0.001 0.001
- link back_right_p2: geometry collision mesh filename=cad_files//simulation//stls//back_right_p2_coarse.stl scale=.001 .001 .001; visual mesh filename=cad_files//simulation//stls//back_right_p2_fine.stl scale=.001 .001 .001
- link back_right_p3: geometry collision mesh filename=cad_files//simulation//stls//back_right_p3_coarse.stl scale=.001 .001 .001; visual mesh filename=cad_files//simulation//stls//back_right_p3_fine.stl scale=.001 .001 .001
- link back_right_p4: geometry collision mesh filename=cad_files//simulation//stls//back_right_p4_coarse.stl scale=.001 .001 .001; visual mesh filename=cad_files//simulation//stls//back_right_p4_fine.stl scale=.001 .001 .001
- link base_plate_bottom: geometry collision mesh filename=cad_files//simulation//stls//base_plate_coarse.stl scale=0.001 0.001 0.001; visual mesh filename=cad_files//simulation//stls//base_plate_fine.stl scale=0.001 0.001 0.001
- link base_plate_top: geometry collision mesh filename=cad_files//simulation//stls//top_plate_coarse.stl scale=0.001 0.001 0.001; visual mesh filename=cad_files//simulation//stls//top_plate_fine.stl scale=0.001 0.001 0.001
- link battery: geometry collision mesh filename=cad_files//simulation//stls//battery_coarse.stl scale=0.001 0.001 0.001; visual mesh filename=cad_files//simulation//stls//battery_fine.stl scale=0.001 0.001 0.001
- link bus: geometry collision mesh filename=cad_files//simulation//stls//bus_coarse.stl scale=.001 .001 .001; visual mesh filename=cad_files//simulation//stls//bus_fine.stl scale=.001 .001 .001
- link conv: geometry collision mesh filename=cad_files//simulation//stls//conv_coarse.stl scale=.001 .001 .001; visual mesh filename=cad_files//simulation//stls//conv_fine.stl scale=.001 .001 .001
- link face: geometry collision mesh filename=cad_files//simulation//stls//face_coarse.stl scale=.001 .001 .001; visual mesh filename=cad_files//simulation//stls//face_fine.stl scale=.001 .001 .001
- link front_left_p1: geometry collision mesh filename=cad_files//simulation//stls//front_left_p1_coarse.stl scale=0.001 0.001 0.001; visual mesh filename=cad_files//simulation//stls//front_left_p1_fine.stl scale=0.001 0.001 0.001
- link front_left_p2: geometry collision mesh filename=cad_files//simulation//stls//front_left_p2_coarse.stl scale=.001 .001 .001; visual mesh filename=cad_files//simulation//stls//front_left_p2_fine.stl scale=.001 .001 .001
- link front_left_p3: geometry collision mesh filename=cad_files//simulation//stls//front_left_p3_coarse.stl scale=.001 .001 .001; visual mesh filename=cad_files//simulation//stls//front_left_p3_fine.stl scale=.001 .001 .001
- link front_left_p4: geometry collision mesh filename=cad_files//simulation//stls//front_left_p4_coarse.stl scale=.001 .001 .001; visual mesh filename=cad_files//simulation//stls//front_left_p4_fine.stl scale=.001 .001 .001
- link front_right_p1: geometry collision mesh filename=cad_files//simulation//stls//front_right_p1_coarse.stl scale=0.001 0.001 0.001; visual mesh filename=cad_files//simulation//stls//front_right_p1_fine.stl scale=0.001 0.001 0.001
- link front_right_p2: geometry collision mesh filename=cad_files//simulation//stls//front_right_p2_coarse.stl scale=.001 .001 .001; visual mesh filename=cad_files//simulation//stls//front_right_p2_fine.stl scale=.001 .001 .001
- link front_right_p3: geometry collision mesh filename=cad_files//simulation//stls//front_right_p3_coarse.stl scale=.001 .001 .001; visual mesh filename=cad_files//simulation//stls//front_right_p3_fine.stl scale=.001 .001 .001
- link front_right_p4: geometry collision mesh filename=cad_files//simulation//stls//front_right_p4_coarse.stl scale=.001 .001 .001; visual mesh filename=cad_files//simulation//stls//front_right_p4_fine.stl scale=.001 .001 .001
- link left_claw: geometry collision mesh filename=cad_files//simulation//stls//left_claw_coarse.stl scale=.001 .001 .001; visual mesh filename=cad_files//simulation//stls//left_claw_fine.stl scale=.001 .001 .001
- link left_leg: geometry collision mesh filename=cad_files//simulation//stls//left_leg_coarse.stl scale=.001 .001 .001; visual mesh filename=cad_files//simulation//stls//left_leg_fine.stl scale=.001 .001 .001
- link pi: geometry collision mesh filename=cad_files//simulation//stls//pi_coarse.stl scale=.001 .001 .001; visual mesh filename=cad_files//simulation//stls//pi_fine.stl scale=.001 .001 .001
- link right_claw: geometry collision mesh filename=cad_files//simulation//stls//right_claw_coarse.stl scale=.001 .001 .001; visual mesh filename=cad_files//simulation//stls//right_claw_fine.stl scale=.001 .001 .001
- link right_leg: geometry collision mesh filename=cad_files//simulation//stls//right_leg_coarse.stl scale=.001 .001 .001; visual mesh filename=cad_files//simulation//stls//right_leg_fine.stl scale=.001 .001 .001

Commit message: Small fix
added slashes to the directories for the urdf, will it work now?

File: sebastian_v2.urdf (robot description, URDF)
Before this commit: robot sebastian, 27 links, 26 joints
Links:
- link back_left_p1: geometry collision mesh filename=//cad_files//simulation//stls//back_left_p1_coarse.stl scale=0.001 0.001 0.001; visual mesh filename=//cad_files//simulation//stls//back_left_p1_fine.stl scale=0.001 0.001 0.001
- link back_left_p2: geometry collision mesh filename=//cad_files//simulation//stls//back_left_p2_coarse.stl scale=.001 .001 .001; visual mesh filename=//cad_files//simulation//stls//back_left_p2_fine.stl scale=.001 .001 .001
- link back_left_p3: geometry collision mesh filename=//cad_files//simulation//stls//back_left_p3_coarse.stl scale=.001 .001 .001; visual mesh filename=//cad_files//simulation//stls//back_left_p3_fine.stl scale=.001 .001 .001
- link back_left_p4: geometry collision mesh filename=//cad_files//simulation//stls//back_left_p4_coarse.stl scale=.001 .001 .001; visual mesh filename=//cad_files//simulation//stls//back_left_p4_fine.stl scale=.001 .001 .001
- link back_right_p1: geometry collision mesh filename=//cad_files//simulation//stls//back_right_p1_coarse.stl scale=0.001 0.001 0.001; visual mesh filename=//cad_files//simulation//stls//back_right_p1_fine.stl scale=0.001 0.001 0.001
- link back_right_p2: geometry collision mesh filename=//cad_files//simulation//stls//back_right_p2_coarse.stl scale=.001 .001 .001; visual mesh filename=//cad_files//simulation//stls//back_right_p2_fine.stl scale=.001 .001 .001
- link back_right_p3: geometry collision mesh filename=//cad_files//simulation//stls//back_right_p3_coarse.stl scale=.001 .001 .001; visual mesh filename=//cad_files//simulation//stls//back_right_p3_fine.stl scale=.001 .001 .001
- link back_right_p4: geometry collision mesh filename=//cad_files//simulation//stls//back_right_p4_coarse.stl scale=.001 .001 .001; visual mesh filename=//cad_files//simulation//stls//back_right_p4_fine.stl scale=.001 .001 .001
- link base_plate_bottom: geometry collision mesh filename=//cad_files//simulation//stls//base_plate_coarse.stl scale=0.001 0.001 0.001; visual mesh filename=//cad_files//simulation//stls//base_plate_fine.stl scale=0.001 0.001 0.001
- link base_plate_top: geometry collision mesh filename=//cad_files//simulation//stls//top_plate_coarse.stl scale=0.001 0.001 0.001; visual mesh filename=//cad_files//simulation//stls//top_plate_fine.stl scale=0.001 0.001 0.001
- link battery: geometry collision mesh filename=//cad_files//simulation//stls//battery_coarse.stl scale=0.001 0.001 0.001; visual mesh filename=//cad_files//simulation//stls//battery_fine.stl scale=0.001 0.001 0.001
- link bus: geometry collision mesh filename=//cad_files//simulation//stls//bus_coarse.stl scale=.001 .001 .001; visual mesh filename=//cad_files//simulation//stls//bus_fine.stl scale=.001 .001 .001
- link conv: geometry collision mesh filename=//cad_files//simulation//stls//conv_coarse.stl scale=.001 .001 .001; visual mesh filename=//cad_files//simulation//stls//conv_fine.stl scale=.001 .001 .001
- link face: geometry collision mesh filename=//cad_files//simulation//stls//face_coarse.stl scale=.001 .001 .001; visual mesh filename=//cad_files//simulation//stls//face_fine.stl scale=.001 .001 .001
- link front_left_p1: geometry collision mesh filename=//cad_files//simulation//stls//front_left_p1_coarse.stl scale=0.001 0.001 0.001; visual mesh filename=//cad_files//simulation//stls//front_left_p1_fine.stl scale=0.001 0.001 0.001
- link front_left_p2: geometry collision mesh filename=//cad_files//simulation//stls//front_left_p2_coarse.stl scale=.001 .001 .001; visual mesh filename=//cad_files//simulation//stls//front_left_p2_fine.stl scale=.001 .001 .001
- link front_left_p3: geometry collision mesh filename=//cad_files//simulation//stls//front_left_p3_coarse.stl scale=.001 .001 .001; visual mesh filename=//cad_files//simulation//stls//front_left_p3_fine.stl scale=.001 .001 .001
- link front_left_p4: geometry collision mesh filename=//cad_files//simulation//stls//front_left_p4_coarse.stl scale=.001 .001 .001; visual mesh filename=//cad_files//simulation//stls//front_left_p4_fine.stl scale=.001 .001 .001
- link front_right_p1: geometry collision mesh filename=//cad_files//simulation//stls//front_right_p1_coarse.stl scale=0.001 0.001 0.001; visual mesh filename=//cad_files//simulation//stls//front_right_p1_fine.stl scale=0.001 0.001 0.001
- link front_right_p2: geometry collision mesh filename=//cad_files//simulation//stls//front_right_p2_coarse.stl scale=.001 .001 .001; visual mesh filename=//cad_files//simulation//stls//front_right_p2_fine.stl scale=.001 .001 .001
- link front_right_p3: geometry collision mesh filename=//cad_files//simulation//stls//front_right_p3_coarse.stl scale=.001 .001 .001; visual mesh filename=//cad_files//simulation//stls//front_right_p3_fine.stl scale=.001 .001 .001
- link front_right_p4: geometry collision mesh filename=//cad_files//simulation//stls//front_right_p4_coarse.stl scale=.001 .001 .001; visual mesh filename=//cad_files//simulation//stls//front_right_p4_fine.stl scale=.001 .001 .001
- link left_claw: geometry collision mesh filename=//cad_files//simulation//stls//left_claw_coarse.stl scale=.001 .001 .001; visual mesh filename=//cad_files//simulation//stls//left_claw_fine.stl scale=.001 .001 .001
- link left_leg: geometry collision mesh filename=//cad_files//simulation//stls//left_leg_coarse.stl scale=.001 .001 .001; visual mesh filename=//cad_files//simulation//stls//left_leg_fine.stl scale=.001 .001 .001
- link pi: geometry collision mesh filename=//cad_files//simulation//stls//pi_coarse.stl scale=.001 .001 .001; visual mesh filename=//cad_files//simulation//stls//pi_fine.stl scale=.001 .001 .001
- link right_claw: geometry collision mesh filename=//cad_files//simulation//stls//right_claw_coarse.stl scale=.001 .001 .001; visual mesh filename=//cad_files//simulation//stls//right_claw_fine.stl scale=.001 .001 .001
- link right_leg: geometry collision mesh filename=//cad_files//simulation//stls//right_leg_coarse.stl scale=.001 .001 .001; visual mesh filename=//cad_files//simulation//stls//right_leg_fine.stl scale=.001 .001 .001

Commit message: stl >> STL
the file ending being lowercase is what fucked me. I hate this.

File: sebastian_v2.urdf (robot description, URDF)
Before this commit: robot sebastian, 27 links, 26 joints
Links:
- link back_left_p1: geometry collision mesh filename=//cad_files//simulation//stls//back_left_p1_coarse.STL scale=0.001 0.001 0.001; visual mesh filename=//cad_files//simulation//stls//back_left_p1_fine.STL scale=0.001 0.001 0.001
- link back_left_p2: geometry collision mesh filename=//cad_files//simulation//stls//back_left_p2_coarse.STL scale=.001 .001 .001; visual mesh filename=//cad_files//simulation//stls//back_left_p2_fine.STL scale=.001 .001 .001
- link back_left_p3: geometry collision mesh filename=//cad_files//simulation//stls//back_left_p3_coarse.STL scale=.001 .001 .001; visual mesh filename=//cad_files//simulation//stls//back_left_p3_fine.STL scale=.001 .001 .001
- link back_left_p4: geometry collision mesh filename=//cad_files//simulation//stls//back_left_p4_coarse.STL scale=.001 .001 .001; visual mesh filename=//cad_files//simulation//stls//back_left_p4_fine.STL scale=.001 .001 .001
- link back_right_p1: geometry collision mesh filename=//cad_files//simulation//stls//back_right_p1_coarse.STL scale=0.001 0.001 0.001; visual mesh filename=//cad_files//simulation//stls//back_right_p1_fine.STL scale=0.001 0.001 0.001
- link back_right_p2: geometry collision mesh filename=//cad_files//simulation//stls//back_right_p2_coarse.STL scale=.001 .001 .001; visual mesh filename=//cad_files//simulation//stls//back_right_p2_fine.STL scale=.001 .001 .001
- link back_right_p3: geometry collision mesh filename=//cad_files//simulation//stls//back_right_p3_coarse.STL scale=.001 .001 .001; visual mesh filename=//cad_files//simulation//stls//back_right_p3_fine.STL scale=.001 .001 .001
- link back_right_p4: geometry collision mesh filename=//cad_files//simulation//stls//back_right_p4_coarse.STL scale=.001 .001 .001; visual mesh filename=//cad_files//simulation//stls//back_right_p4_fine.STL scale=.001 .001 .001
- link base_plate_bottom: geometry collision mesh filename=//cad_files//simulation//stls//base_plate_coarse.STL scale=0.001 0.001 0.001; visual mesh filename=//cad_files//simulation//stls//base_plate_fine.STL scale=0.001 0.001 0.001
- link base_plate_top: geometry collision mesh filename=//cad_files//simulation//stls//top_plate_coarse.STL scale=0.001 0.001 0.001; visual mesh filename=//cad_files//simulation//stls//top_plate_fine.STL scale=0.001 0.001 0.001
- link battery: geometry collision mesh filename=//cad_files//simulation//stls//battery_coarse.STL scale=0.001 0.001 0.001; visual mesh filename=//cad_files//simulation//stls//battery_fine.STL scale=0.001 0.001 0.001
- link bus: geometry collision mesh filename=//cad_files//simulation//stls//bus_coarse.STL scale=.001 .001 .001; visual mesh filename=//cad_files//simulation//stls//bus_fine.STL scale=.001 .001 .001
- link conv: geometry collision mesh filename=//cad_files//simulation//stls//conv_coarse.STL scale=.001 .001 .001; visual mesh filename=//cad_files//simulation//stls//conv_fine.STL scale=.001 .001 .001
- link face: geometry collision mesh filename=//cad_files//simulation//stls//face_coarse.STL scale=.001 .001 .001; visual mesh filename=//cad_files//simulation//stls//face_fine.STL scale=.001 .001 .001
- link front_left_p1: geometry collision mesh filename=//cad_files//simulation//stls//front_left_p1_coarse.STL scale=0.001 0.001 0.001; visual mesh filename=//cad_files//simulation//stls//front_left_p1_fine.STL scale=0.001 0.001 0.001
- link front_left_p2: geometry collision mesh filename=//cad_files//simulation//stls//front_left_p2_coarse.STL scale=.001 .001 .001; visual mesh filename=//cad_files//simulation//stls//front_left_p2_fine.STL scale=.001 .001 .001
- link front_left_p3: geometry collision mesh filename=//cad_files//simulation//stls//front_left_p3_coarse.STL scale=.001 .001 .001; visual mesh filename=//cad_files//simulation//stls//front_left_p3_fine.STL scale=.001 .001 .001
- link front_left_p4: geometry collision mesh filename=//cad_files//simulation//stls//front_left_p4_coarse.STL scale=.001 .001 .001; visual mesh filename=//cad_files//simulation//stls//front_left_p4_fine.STL scale=.001 .001 .001
- link front_right_p1: geometry collision mesh filename=//cad_files//simulation//stls//front_right_p1_coarse.STL scale=0.001 0.001 0.001; visual mesh filename=//cad_files//simulation//stls//front_right_p1_fine.STL scale=0.001 0.001 0.001
- link front_right_p2: geometry collision mesh filename=//cad_files//simulation//stls//front_right_p2_coarse.STL scale=.001 .001 .001; visual mesh filename=//cad_files//simulation//stls//front_right_p2_fine.STL scale=.001 .001 .001
- link front_right_p3: geometry collision mesh filename=//cad_files//simulation//stls//front_right_p3_coarse.STL scale=.001 .001 .001; visual mesh filename=//cad_files//simulation//stls//front_right_p3_fine.STL scale=.001 .001 .001
- link front_right_p4: geometry collision mesh filename=//cad_files//simulation//stls//front_right_p4_coarse.STL scale=.001 .001 .001; visual mesh filename=//cad_files//simulation//stls//front_right_p4_fine.STL scale=.001 .001 .001
- link left_claw: geometry collision mesh filename=//cad_files//simulation//stls//left_claw_coarse.STL scale=.001 .001 .001; visual mesh filename=//cad_files//simulation//stls//left_claw_fine.STL scale=.001 .001 .001
- link left_leg: geometry collision mesh filename=//cad_files//simulation//stls//left_leg_coarse.STL scale=.001 .001 .001; visual mesh filename=//cad_files//simulation//stls//left_leg_fine.STL scale=.001 .001 .001
- link pi: geometry collision mesh filename=//cad_files//simulation//stls//pi_coarse.STL scale=.001 .001 .001; visual mesh filename=//cad_files//simulation//stls//pi_fine.STL scale=.001 .001 .001
- link right_claw: geometry collision mesh filename=//cad_files//simulation//stls//right_claw_coarse.STL scale=.001 .001 .001; visual mesh filename=//cad_files//simulation//stls//right_claw_fine.STL scale=.001 .001 .001
- link right_leg: geometry collision mesh filename=//cad_files//simulation//stls//right_leg_coarse.STL scale=.001 .001 .001; visual mesh filename=//cad_files//simulation//stls//right_leg_fine.STL scale=.001 .001 .001

Commit message: updated urdf, investigating
updated urdf model since back legs aren't going to be used, also looking into whether I should shift to velocity control since my motors won't be reading xyz position

File: sebastian_v2.urdf (robot description, URDF)
Before this commit: robot sebastian, 27 links, 26 joints
Links:
- removed link left_leg
- removed link right_leg
Joints:
- removed joint base_bottom_to_left_leg
- removed joint base_bottom_to_right_leg
