Commit message: made small changes to a few things
slightly upped the range of the leg ends, added moving averages to plotter.py, toyed with deviation and yaw reward

File: sebastian_v3.urdf (robot description, URDF)
Before this commit: robot sebastian, 23 links, 22 joints
Joints:
- joint back_left_p3p4: limit lower=-1.5708 upper=.4 effort=1000 velocity=1 -> lower=-1.5708 upper=.5 effort=1000 velocity=1
- joint back_right_p3p4: limit lower=-.4 upper=1.5708 effort=1000 velocity=1 -> lower=-.5 upper=1.5708 effort=1000 velocity=1
- joint front_left_p3p4: limit lower=-1.5708 upper=.4 effort=1000 velocity=1 -> lower=-1.5708 upper=.5 effort=1000 velocity=1
- joint front_right_p3p4: limit lower=-.4 upper=1.5708 effort=1000 velocity=1 -> lower=-.5 upper=1.5708 effort=1000 velocity=1

Commit message: reoriented robot to more manageable start position
Calibrating the physical robot motor positions is still a giant pain since I don't know a good way to do it, so I'm initializing the robot in a very angular way to make it easier on me - more parallel and perpendicular arrangements for the legs. Also did some reorganizing and updated the URDF to match the new config, will need to retrain on this model now. First, need to update the leg ranges again.

File: sebastian_v3.urdf (robot description, URDF)
Before this commit: robot sebastian, 23 links, 22 joints
Joints:
- joint back_left_p2p3: origin xyz=.06069 0.018 -0.00696 -> xyz=0.04590633696 0.0435860972 -0.00696
- joint back_left_p3p4: origin xyz=0.06704 -0.00023 -0.01303 -> xyz=0.0597405058 0.0304179711 -0.01303
- joint back_right_p2p3: origin xyz=-.06069 -0.018 -0.00696 -> xyz=-0.0622470528 0.0115074672 -0.00696
- joint back_right_p3p4: origin xyz=-0.06704 -0.00023 -0.01303 -> xyz=-0.0597276669 0.0304431735 -0.01303
- joint front_left_p2p3: origin xyz=.06069 0.018 -0.00696 -> xyz=0.0632262127 -0.0034342938 -0.0069580693
- joint front_left_p3p4: origin xyz=0.06704 -0.00023 -0.01303 -> xyz=0.0632567046 -0.0221984307 -0.0130277886
- joint front_right_p2p3: origin xyz=-.06069 -0.018 -0.00696 -> xyz=-0.0515981457 -0.0367139955 -0.0069580693
- joint front_right_p3p4: origin xyz=-0.06704 -0.00023 -0.01303 -> xyz=-0.0632660647 -0.0221717401 -0.01303

Commit message: need to update joint axes
for whatever reason the joint axes are crooked for p2p3 and maybe p3p4, will need to take a look on Amelia to see how to fix it

File: sebastian_v3.urdf (robot description, URDF)
Before this commit: robot sebastian, 23 links, 22 joints
Joints:
- joint back_left_p1p2: limit lower=0.0 upper=0.548 effort=1000.0 velocity=1 -> lower=-1 upper=0.75 effort=1000.0 velocity=1
- joint back_right_p1p2: limit lower=0.0 upper=0.548 effort=1000.0 velocity=1 -> lower=-0.75 upper=1 effort=1000.0 velocity=1
- joint front_left_p1p2: limit lower=0.0 upper=0.548 effort=1000.0 velocity=1 -> lower=-1 upper=0.75 effort=1000.0 velocity=1
- joint front_right_p1p2: limit lower=0.0 upper=0.548 effort=1000.0 velocity=1 -> lower=-0.75 upper=1 effort=1000.0 velocity=1

Commit message: corrected joint positions, updated ranges
Noticed that the joint axes were messed up, so I fixed them. Also updated the leg ranges. Finally, I can rerun the training on colab

File: sebastian_v3.urdf (robot description, URDF)
Before this commit: robot sebastian, 23 links, 22 joints
Joints:
- joint back_left_p1p2: limit lower=-1 upper=0.75 effort=1000.0 velocity=1 -> lower=-0.6 upper=0.8 effort=1000.0 velocity=1
- joint back_left_p2p3: limit lower=-1.5708 upper=.9 effort=1000 velocity=1 -> lower=-.9 upper=.9 effort=1000 velocity=1; origin xyz=0.04590633696 0.0435860972 -0.00696 -> xyz=0.04590633696 0.0435860972 -0.00696 rpy=0 0 0.47133
- joint back_left_p3p4: limit lower=-1.5708 upper=.5 effort=1000 velocity=1 -> lower=-1.2 upper=.8 effort=1000 velocity=1; origin xyz=0.0597405058 0.0304179711 -0.01303 -> xyz=0.06704 -0.00023 -0.01303
- joint back_right_p1p2: limit lower=-0.75 upper=1 effort=1000.0 velocity=1 -> lower=-0.6 upper=0.8 effort=1000.0 velocity=1
- joint back_right_p2p3: limit lower=-.9 upper=1.5708 effort=1000 velocity=1 -> lower=-.9 upper=.9 effort=1000 velocity=1; origin xyz=-0.0622470528 0.0115074672 -0.00696 -> xyz=-0.0622470528 0.0115074672 -0.00696 rpy=0 0 -0.471239
- joint back_right_p3p4: limit lower=-.5 upper=1.5708 effort=1000 velocity=1 -> lower=-1.2 upper=.8 effort=1000 velocity=1; origin xyz=-0.0597276669 0.0304431735 -0.01303 -> xyz=-0.06704 -0.00023 -0.01303
- joint front_left_p1p2: limit lower=-1 upper=0.75 effort=1000.0 velocity=1 -> lower=-0.8 upper=0.6 effort=1000.0 velocity=1
- joint front_left_p2p3: limit lower=-1.5708 upper=.9 effort=1000 velocity=1 -> lower=-.9 upper=.9 effort=1000 velocity=1; origin xyz=0.0632262127 -0.0034342938 -0.0069580693 -> xyz=0.0632262127 -0.0034342938 -0.0069580693 rpy=0 0 2.804
- joint front_left_p3p4: limit lower=-1.5708 upper=.5 effort=1000 velocity=1 -> lower=-0.8 upper=1.2 effort=1000 velocity=1; origin xyz=0.0632567046 -0.0221984307 -0.0130277886 -> xyz=-0.06704 -0.00023 -0.01303 rpy=0 0 0
- joint front_right_p1p2: limit lower=-0.75 upper=1 effort=1000.0 velocity=1 -> lower=-0.8 upper=0.6 effort=1000.0 velocity=1
- joint front_right_p2p3: limit lower=-.9 upper=1.5708 effort=1000 velocity=1 -> lower=-.9 upper=0.9 effort=1000 velocity=1; origin xyz=-0.0515981457 -0.0367139955 -0.0069580693 -> xyz=-0.0515981457 -0.0367139955 -0.0069580693 rpy=0 0 0.3374
- joint front_right_p3p4: limit lower=-.5 upper=1.5708 effort=1000 velocity=1 -> lower=-.8 upper=1.2 effort=1000 velocity=1; origin xyz=-0.0632660647 -0.0221717401 -0.01303 -> xyz=-0.06704 -0.00023 -0.01303
